Commit message: My_robot personally edited

File: src/my_robot/urdf/my_robot.xacro (robot description, xacro)
@@ -8,8 +8,9 @@
     <child link="chassis" />
   </joint>
+<!-- Chassis -->
   <link name='chassis'>
     <pose>0 0 0.1 0 0 0</pose>
     <inertial>
-      <mass value="15.0"/>
+      <mass value="10.0"/>
       <origin xyz="0.0 0 0" rpy=" 0 0 0"/>
       <inertia
@@ -22,5 +23,5 @@
       <origin xyz="0 0 0" rpy=" 0 0 0"/>
       <geometry>
-        <box size=".4 .2 .1"/>
+        <box size=".5 .3 .2"/>
       </geometry>
     </collision>
@@ -28,37 +29,31 @@
       <origin xyz="0 0 0" rpy=" 0 0 0"/>
       <geometry>
-        <box size=".4 .2 .1"/>
-      </geometry>
-    </visual>
-    <collision name='back_caster_collision'>
-      <origin xyz="-0.15 0 -0.05" rpy=" 0 0 0"/>
+        <box size=".4 .2 .2"/>
+      </geometry>
+      <material name="red">
+		<color rgba= "1 0 0 0.2"/>
+      </material>
+    </visual>
+    <collision name='front_caster_collision'>
+      <origin xyz="0.15 0 -0.1" rpy=" 0 0 0"/>
       <geometry>
         <sphere radius="0.0499"/>
       </geometry>
     </collision>
-    <visual name='back_caster_visual'>
-      <origin xyz="-0.15 0 -0.05" rpy=" 0 0 0"/>
+    <visual name='front_caster_visual'>
+      <origin xyz="0.15 0 -0.1" rpy=" 0 0 0"/>
       <geometry>
         <sphere radius="0.05"/>
       </geometry>
-    </visual>
-    <collision name='front_caster_collision'>
-      <origin xyz="0.15 0 -0.05" rpy=" 0 0 0"/>
-      <geometry>
-        <sphere radius="0.0499"/>
-      </geometry>
-    </collision>
-    <visual name='front_caster_visual'>
-      <origin xyz="0.15 0 -0.05" rpy=" 0 0 0"/>
-      <geometry>
-        <sphere radius="0.05"/>
-      </geometry>
-    </visual>
-  </link>
+	<material name="black">
+		<color rgba= "0 0 0 0.5"/>
+      </material>
+    </visual>
+  </link>
+<!-- Left Wheel -->
   <link name='left_wheel'>
-    <pose>0 0 0.1 0 0 0</pose>
     <inertial>
       <mass value="5.0"/>
-      <origin xyz="0.0 0 0" rpy=" 0 1.5707 1.5707"/>
+      <origin xyz="0 0 0" rpy=" 0 1.5707 1.5707"/>
       <inertia
           ixx="0.1" ixy="0" ixz="0"
@@ -78,8 +73,11 @@
         <cylinder radius="0.1" length="0.05"/>
       </geometry>
+      <material name="black">
+		<color rgba= "0 0 0 0.5"/>
+      </material>
     </visual>
   </link>
   <joint type="continuous" name="left_wheel_hinge">
-    <origin xyz="0 0.15 0" rpy="0 0 0"/>
+    <origin xyz="-0.1 0.15 -0.05" rpy="0 0 0"/>
     <child link="left_wheel"/>
     <parent link="chassis"/>
@@ -88,6 +86,6 @@
     <dynamics damping="1.0" friction="1.0"/>
   </joint>
+<!-- Right Wheel -->
   <link name='right_wheel'>
-    <pose>0 0 0.1 0 0 0</pose>
     <inertial>
       <mass value="5.0"/>
@@ -110,8 +108,11 @@
         <cylinder radius="0.1" length="0.05"/>
       </geometry>
+	<material name="black">
+		<color rgba= "0 0 0 0.5"/>
+      </material>
     </visual>
   </link>
   <joint type="continuous" name="right_wheel_hinge">
-    <origin xyz="0 -0.15 0" rpy="0 0 0"/>
+    <origin xyz="-0.1 -0.15 -0.05" rpy="0 0 0"/>
     <child link="right_wheel"/>
     <parent link="chassis"/>
@@ -120,4 +121,5 @@
     <dynamics damping="1.0" friction="1.0"/>
   </joint>
+<!-- Camera -->
   <link name='camera'>
     <pose>0 0 0.1 0 0 0</pose>
@@ -143,4 +145,7 @@
         <box size="0.05 0.05 0.05"/>
         <box_inertia m="0.1" x="0.05" y="0.05" z="0.05"/>
+	<material name="white">
+		<color rgba= "1 1 1 0.5"/>
+         </material>
       </geometry>
     </visual>
@@ -154,4 +159,5 @@
     <dynamics damping="1.0" friction="1.0"/>
   </joint>
+<!-- Lidar -->
   <link name='hokuyo'>
     <pose>0 0 0.1 0 0 0</pose>
@@ -179,5 +185,5 @@
   </link>
   <joint type="fixed" name="hokuyo_joint">
-    <origin xyz="0.15 0 0.1" rpy="0 0 0"/>
+    <origin xyz="0.15 0 0.13" rpy="0 0 0"/>
     <child link="hokuyo"/>
     <parent link="chassis"/>
@@ -186,3 +192,19 @@
     <dynamics damping="1.0" friction="1.0"/>
   </joint>
+<!-- Color -->
+  <gazebo reference="chassis">
+    <material>Gazebo/Red</material>
+  </gazebo>
+  <gazebo reference="left_wheel">
+    <material>Gazebo/DarkGrey</material>
+  </gazebo>
+  <gazebo reference="right_wheel">
+    <material>Gazebo/DarkGrey</material>
+  </gazebo>
+  <gazebo reference="hokuyo">
+    <material>Gazebo/DarkGrey</material>
+  </gazebo>
+  <gazebo reference="camera">
+    <material>Gazebo/White</material>
+  </gazebo>
 </robot>

Commit message: my_robot changed, process_image routine changed to a better center pixel detection, my_robot urdf changed

File: src/my_robot/urdf/my_robot.xacro (robot description, xacro)
@@ -8,9 +8,8 @@
     <child link="chassis" />
   </joint>
-<!-- Chassis -->
   <link name='chassis'>
     <pose>0 0 0.1 0 0 0</pose>
     <inertial>
-      <mass value="10.0"/>
+      <mass value="15.0"/>
       <origin xyz="0.0 0 0" rpy=" 0 0 0"/>
       <inertia
@@ -23,5 +22,5 @@
       <origin xyz="0 0 0" rpy=" 0 0 0"/>
       <geometry>
-        <box size=".5 .3 .2"/>
+        <box size=".4 .25 .1"/>
       </geometry>
     </collision>
@@ -29,12 +28,21 @@
       <origin xyz="0 0 0" rpy=" 0 0 0"/>
       <geometry>
-        <box size=".4 .2 .2"/>
-      </geometry>
-      <material name="red">
-		<color rgba= "1 0 0 0.2"/>
-      </material>
+        <box size=".4 .25 .1"/>
+      </geometry>
+    </visual>
+	<collision name='back_caster_collision'>
+      <origin xyz="-0.15 0 -0.05" rpy=" 0 0 0"/>
+      <geometry>
+        <sphere radius="0.0499"/>
+      </geometry>
+    </collision>
+    <visual name='back_caster_visual'>
+      <origin xyz="-0.15 0 -0.05" rpy=" 0 0 0"/>
+      <geometry>
+        <sphere radius="0.05"/>
+      </geometry>
     </visual>
     <collision name='front_caster_collision'>
-      <origin xyz="0.15 0 -0.1" rpy=" 0 0 0"/>
+      <origin xyz="0.15 0 -0.05" rpy=" 0 0 0"/>
       <geometry>
         <sphere radius="0.0499"/>
@@ -42,18 +50,15 @@
     </collision>
     <visual name='front_caster_visual'>
-      <origin xyz="0.15 0 -0.1" rpy=" 0 0 0"/>
+      <origin xyz="0.15 0 -0.05" rpy=" 0 0 0"/>
       <geometry>
         <sphere radius="0.05"/>
       </geometry>
-	<material name="black">
-		<color rgba= "0 0 0 0.5"/>
-      </material>
-    </visual>
-  </link>
-<!-- Left Wheel -->
+    </visual>
+  </link>
   <link name='left_wheel'>
+    <pose>0 0 0.1 0 0 0</pose>
     <inertial>
       <mass value="5.0"/>
-      <origin xyz="0 0 0" rpy=" 0 1.5707 1.5707"/>
+      <origin xyz="0.0 0 0" rpy=" 0 1.5707 1.5707"/>
       <inertia
           ixx="0.1" ixy="0" ixz="0"
@@ -65,5 +70,5 @@
       <origin xyz="0 0 0" rpy=" 0 1.5707 1.5707"/>
       <geometry>
-        <cylinder radius="0.1" length="0.05"/>
+        <cylinder radius="0.1" length="0.1"/>
       </geometry>
     </collision>
@@ -71,13 +76,10 @@
       <origin xyz="0 0 0" rpy=" 0 1.5707 1.5707"/>
       <geometry>
-        <cylinder radius="0.1" length="0.05"/>
-      </geometry>
-      <material name="black">
-		<color rgba= "0 0 0 0.5"/>
-      </material>
+        <cylinder radius="0.1" length="0.1"/>
+      </geometry>
     </visual>
   </link>
   <joint type="continuous" name="left_wheel_hinge">
-    <origin xyz="-0.1 0.15 -0.05" rpy="0 0 0"/>
+    <origin xyz="0 0.2 0" rpy="0 0 0"/>
     <child link="left_wheel"/>
     <parent link="chassis"/>
@@ -86,6 +88,6 @@
     <dynamics damping="1.0" friction="1.0"/>
   </joint>
-<!-- Right Wheel -->
   <link name='right_wheel'>
+    <pose>0 0 0.1 0 0 0</pose>
     <inertial>
       <mass value="5.0"/>
@@ -100,5 +102,5 @@
       <origin xyz="0 0 0" rpy=" 0 1.5707 1.5707"/>
       <geometry>
-        <cylinder radius="0.1" length="0.05"/>
+        <cylinder radius="0.1" length="0.1"/>
       </geometry>
     </collision>
@@ -106,13 +108,10 @@
       <origin xyz="0 0 0" rpy=" 0 1.5707 1.5707"/>
       <geometry>
-        <cylinder radius="0.1" length="0.05"/>
-      </geometry>
-	<material name="black">
-		<color rgba= "0 0 0 0.5"/>
-      </material>
+        <cylinder radius="0.1" length="0.1"/>
+      </geometry>
     </visual>
   </link>
   <joint type="continuous" name="right_wheel_hinge">
-    <origin xyz="-0.1 -0.15 -0.05" rpy="0 0 0"/>
+    <origin xyz="0 -0.2 0" rpy="0 0 0"/>
     <child link="right_wheel"/>
     <parent link="chassis"/>
@@ -121,5 +120,4 @@
     <dynamics damping="1.0" friction="1.0"/>
   </joint>
-<!-- Camera -->
   <link name='camera'>
     <pose>0 0 0.1 0 0 0</pose>
@@ -145,7 +143,4 @@
         <box size="0.05 0.05 0.05"/>
         <box_inertia m="0.1" x="0.05" y="0.05" z="0.05"/>
-	<material name="white">
-		<color rgba= "1 1 1 0.5"/>
-         </material>
       </geometry>
     </visual>
@@ -159,5 +154,4 @@
     <dynamics damping="1.0" friction="1.0"/>
   </joint>
-<!-- Lidar -->
   <link name='hokuyo'>
     <pose>0 0 0.1 0 0 0</pose>
@@ -185,5 +179,5 @@
   </link>
   <joint type="fixed" name="hokuyo_joint">
-    <origin xyz="0.15 0 0.13" rpy="0 0 0"/>
+    <origin xyz="0.15 0 0.1" rpy="0 0 0"/>
     <child link="hokuyo"/>
     <parent link="chassis"/>

Commit message: SLAM added through rtabmap, rgb-d camera added

File: src/my_robot/urdf/my_robot.xacro (robot description, xacro)
@@ -154,4 +154,11 @@
     <dynamics damping="1.0" friction="1.0"/>
   </joint>
+  <joint name="camera_optical_joint" type="fixed">
+    <origin xyz="0 0 0" rpy="-1.5707 0 -1.5707"/>
+    <parent link="camera"/>
+    <child link="camera_link_optical"/>
+  </joint>
+  <link name="camera_link_optical">
+  </link>
   <link name='hokuyo'>
     <pose>0 0 0.1 0 0 0</pose>
